File: voltage_regulators.sch (KiCad schematic (older format))
At the start: 18 parts

Commit message: Annotate schematic symbols
Parts:
- gave numbers to parts that had none: 18
Changed lines of the file:
@@
 $EndDescr
 $Comp
-L Connector_Generic:Conn_01x02 J?
+L Connector_Generic:Conn_01x02 J1
 U 1 1 60B221B5
 P 2150 1950
-F 0 "J?" H 2068 2167 50  0000 C CNN
+F 0 "J1" H 2068 2167 50  0000 C CNN
 F 1 "Conn_01x02" H 2068 2076 50  0000 C CNN
 F 2 "" H 2150 1950 50  0001 C CNN
@@
 $EndComp
 $Comp
-L Connector_Generic:Conn_01x02 J?
+L Connector_Generic:Conn_01x02 J2
 U 1 1 60B238B2
 P 2150 2400
-F 0 "J?" H 2068 2617 50  0000 C CNN
+F 0 "J2" H 2068 2617 50  0000 C CNN
 F 1 "Conn_01x02" H 2068 2526 50  0000 C CNN
 F 2 "" H 2150 2400 50  0001 C CNN
@@
 $EndComp
 $Comp
-L Switch:SW_SPDT SW?
+L Switch:SW_SPDT SW1
 U 1 1 60B247FD
 P 2800 1950
-F 0 "SW?" H 2800 2235 50  0000 C CNN
+F 0 "SW1" H 2800 2235 50  0000 C CNN
 F 1 "SW_SPDT" H 2800 2144 50  0000 C CNN
 F 2 "" H 2800 1950 50  0001 C CNN
@@
 $EndComp
 $Comp
-L Transistor_FET:FDS9435A Q?
+L Transistor_FET:FDS9435A Q1
 U 1 1 60B277D5
 P 3300 2150
-F 0 "Q?" V 3642 2150 50  0000 C CNN
+F 0 "Q1" V 3642 2150 50  0000 C CNN
 F 1 "FDS4141" V 3551 2150 50  0000 C CNN
 F 2 "Package_SO:SOIC-8_3.9x4.9mm_P1.27mm" H 3500 2075 50  0001 L CIN
@@
 $EndComp
 $Comp
-L Device:R R?
+L Device:R R1
 U 1 1 60B29A16
 P 3600 2300
-F 0 "R?" H 3670 2346 50  0000 L CNN
+F 0 "R1" H 3670 2346 50  0000 L CNN
 F 1 "1k" H 3670 2255 50  0000 L CNN
 F 2 "" V 3530 2300 50  0001 C CNN
@@
 $EndComp
 $Comp
-L Device:R R?
+L Device:R R2
 U 1 1 60B2D1FC
 P 3600 2650
-F 0 "R?" H 3670 2696 50  0000 L CNN
+F 0 "R2" H 3670 2696 50  0000 L CNN
 F 1 "1k" H 3670 2605 50  0000 L CNN
 F 2 "" V 3530 2650 50  0001 C CNN
@@
 $EndComp
 $Comp
-L Device:LED D?
+L Device:LED D1
 U 1 1 60B302CE
 P 3600 3000
-F 0 "D?" V 3639 2882 50  0000 R CNN
+F 0 "D1" V 3639 2882 50  0000 R CNN
 F 1 "RED LED" V 3548 2882 50  0000 R CNN
 F 2 "" H 3600 3000 50  0001 C CNN
@@
 $EndComp
 $Comp
-L power:+BATT #PWR?
+L power:+BATT #PWR03
 U 1 1 60B318F0
 P 3600 1750
-F 0 "#PWR?" H 3600 1600 50  0001 C CNN
+F 0 "#PWR03" H 3600 1600 50  0001 C CNN
 F 1 "+BATT" H 3615 1923 50  0000 C CNN
 F 2 "" H 3600 1750 50  0001 C CNN
@@
 $EndComp
 $Comp
-L power:+BATT #PWR?
+L power:+BATT #PWR05
 U 1 1 60B33BB0
 P 5050 1750
-F 0 "#PWR?" H 5050 1600 50  0001 C CNN
+F 0 "#PWR05" H 5050 1600 50  0001 C CNN
 F 1 "+BATT" H 5065 1923 50  0000 C CNN
 F 2 "" H 5050 1750 50  0001 C CNN
@@
 $EndComp
 $Comp
-L Device:C C?
+L Device:C C1
 U 1 1 60B33CDA
 P 5050 2600
-F 0 "C?" H 5165 2646 50  0000 L CNN
+F 0 "C1" H 5165 2646 50  0000 L CNN
 F 1 "4u7" H 5165 2555 50  0000 L CNN
 F 2 "" H 5088 2450 50  0001 C CNN
@@
 $EndComp
 $Comp
-L Device:C C?
+L Device:C C2
 U 1 1 60B34B48
 P 5450 2600
-F 0 "C?" H 5565 2646 50  0000 L CNN
+F 0 "C2" H 5565 2646 50  0000 L CNN
 F 1 "100n" H 5565 2555 50  0000 L CNN
 F 2 "" H 5488 2450 50  0001 C CNN
@@
 $EndComp
 $Comp
-L Regulator_Switching:ST1S10PHR U?
+L Regulator_Switching:ST1S10PHR U1
 U 1 1 60B35791
 P 6400 2150
-F 0 "U?" H 6400 2492 50  0000 C CNN
+F 0 "U1" H 6400 2492 50  0000 C CNN
 F 1 "ST1S10PHR" H 6400 2401 50  0000 C CNN
 F 2 "Package_SO:TI_SO-PowerPAD-8" H 6525 1800 50  0001 L CIN
@@
 $EndComp
 $Comp
-L Device:L L?
+L Device:L L1
 U 1 1 60B37251
 P 7100 2050
-F 0 "L?" V 7290 2050 50  0000 C CNN
+F 0 "L1" V 7290 2050 50  0000 C CNN
 F 1 "3u3" V 7199 2050 50  0000 C CNN
 F 2 "" H 7100 2050 50  0001 C CNN
@@
 $EndComp
 $Comp
-L Device:R R?
+L Device:R R3
 U 1 1 60B382AA
 P 7350 2300
-F 0 "R?" H 7420 2346 50  0000 L CNN
+F 0 "R3" H 7420 2346 50  0000 L CNN
 F 1 "100k" H 7420 2255 50  0000 L CNN
 F 2 "" V 7280 2300 50  0001 C CNN
@@
 $EndComp
 $Comp
-L Device:R R?
+L Device:R R4
 U 1 1 60B38FE8
 P 7350 2650
-F 0 "R?" H 7420 2696 50  0000 L CNN
+F 0 "R4" H 7420 2696 50  0000 L CNN
 F 1 "5k1" H 7420 2605 50  0000 L CNN
 F 2 "" V 7280 2650 50  0001 C CNN
@@
 $EndComp
 $Comp
-L Device:R R?
+L Device:R R5
 U 1 1 60B399B5
 P 7350 3050
-F 0 "R?" H 7420 3096 50  0000 L CNN
+F 0 "R5" H 7420 3096 50  0000 L CNN
 F 1 "20k" H 7420 3005 50  0000 L CNN
 F 2 "" V 7280 3050 50  0001 C CNN
@@
 $EndComp
 $Comp
-L Device:C C?
+L Device:C C3
 U 1 1 60B3A425
 P 7750 2300
-F 0 "C?" H 7865 2346 50  0000 L CNN
+F 0 "C3" H 7865 2346 50  0000 L CNN
 F 1 "22u" H 7865 2255 50  0000 L CNN
 F 2 "" H 7788 2150 50  0001 C CNN
@@
 $EndComp
 $Comp
-L power:+5V #PWR?
+L power:+5V #PWR015
 U 1 1 60B3BAD6
 P 7750 1750
-F 0 "#PWR?" H 7750 1600 50  0001 C CNN
+F 0 "#PWR015" H 7750 1600 50  0001 C CNN
 F 1 "+5V" H 7765 1923 50  0000 C CNN
 F 2 "" H 7750 1750 50  0001 C CNN
@@
 $EndComp
 $Comp
-L power:+5V #PWR?
+L power:+5V #PWR07
 U 1 1 60B3D7D9
 P 5050 4200
-F 0 "#PWR?" H 5050 4050 50  0001 C CNN
+F 0 "#PWR07" H 5050 4050 50  0001 C CNN
 F 1 "+5V" H 5065 4373 50  0000 C CNN
 F 2 "" H 5050 4200 50  0001 C CNN
@@
 $EndComp
 $Comp
-L Device:CP C?
+L Device:CP C4
 U 1 1 60B3E4FF
 P 5050 4550
-F 0 "C?" H 5168 4596 50  0000 L CNN
+F 0 "C4" H 5168 4596 50  0000 L CNN
 F 1 "10u" H 5168 4505 50  0000 L CNN
 F 2 "" H 5088 4400 50  0001 C CNN
@@
 $EndComp
 $Comp
-L Regulator_Linear:LM1117-3.3 U?
+L Regulator_Linear:LM1117-3.3 U2
 U 1 1 60B404E7
 P 5750 4300
-F 0 "U?" H 5750 4542 50  0000 C CNN
+F 0 "U2" H 5750 4542 50  0000 C CNN
 F 1 "LM1117-3.3" H 5750 4451 50  0000 C CNN
 F 2 "" H 5750 4300 50  0001 C CNN
@@
 $EndComp
 $Comp
-L Device:CP C?
+L Device:CP C5
 U 1 1 60B41B3F
 P 6450 4550
-F 0 "C?" H 6568 4596 50  0000 L CNN
+F 0 "C5" H 6568 4596 50  0000 L CNN
 F 1 "10u" H 6568 4505 50  0000 L CNN
 F 2 "" H 6488 4400 50  0001 C CNN
@@
 $EndComp
 $Comp
-L power:+3V3 #PWR?
+L power:+3V3 #PWR012
 U 1 1 60B42C58
 P 6450 4200
-F 0 "#PWR?" H 6450 4050 50  0001 C CNN
+F 0 "#PWR012" H 6450 4050 50  0001 C CNN
 F 1 "+3V3" H 6465 4373 50  0000 C CNN
 F 2 "" H 6450 4200 50  0001 C CNN
@@
 $EndComp
 $Comp
-L power:GND #PWR?
+L power:GND #PWR01
 U 1 1 60B446B0
 P 2450 2650
-F 0 "#PWR?" H 2450 2400 50  0001 C CNN
+F 0 "#PWR01" H 2450 2400 50  0001 C CNN
 F 1 "GND" H 2455 2477 50  0000 C CNN
 F 2 "" H 2450 2650 50  0001 C CNN
@@
 $EndComp
 $Comp
-L power:GND #PWR?
+L power:GND #PWR02
 U 1 1 60B46A1B
 P 3300 2650
-F 0 "#PWR?" H 3300 2400 50  0001 C CNN
+F 0 "#PWR02" H 3300 2400 50  0001 C CNN
 F 1 "GND" H 3305 2477 50  0000 C CNN
 F 2 "" H 3300 2650 50  0001 C CNN
@@
 $EndComp
 $Comp
-L power:GND #PWR?
+L power:GND #PWR04
 U 1 1 60B470DF
 P 3600 3250
-F 0 "#PWR?" H 3600 3000 50  0001 C CNN
+F 0 "#PWR04" H 3600 3000 50  0001 C CNN
 F 1 "GND" H 3605 3077 50  0000 C CNN
 F 2 "" H 3600 3250 50  0001 C CNN
@@
 $EndComp
 $Comp
-L power:GND #PWR?
+L power:GND #PWR06
 U 1 1 60B4757A
 P 5050 2850
-F 0 "#PWR?" H 5050 2600 50  0001 C CNN
+F 0 "#PWR06" H 5050 2600 50  0001 C CNN
 F 1 "GND" H 5055 2677 50  0000 C CNN
 F 2 "" H 5050 2850 50  0001 C CNN
@@
 $EndComp
 $Comp
-L power:GND #PWR?
+L power:GND #PWR09
 U 1 1 60B47C68
 P 5450 2850
-F 0 "#PWR?" H 5450 2600 50  0001 C CNN
+F 0 "#PWR09" H 5450 2600 50  0001 C CNN
 F 1 "GND" H 5455 2677 50  0000 C CNN
 F 2 "" H 5450 2850 50  0001 C CNN
@@
 $EndComp
 $Comp
-L power:GND #PWR?
+L power:GND #PWR011
 U 1 1 60B487B5
 P 5850 2850
-F 0 "#PWR?" H 5850 2600 50  0001 C CNN
+F 0 "#PWR011" H 5850 2600 50  0001 C CNN
 F 1 "GND" H 5855 2677 50  0000 C CNN
 F 2 "" H 5850 2850 50  0001 C CNN
@@
 $EndComp
 $Comp
-L power:GND #PWR?
+L power:GND #PWR014
 U 1 1 60B497AD
 P 7350 3300
-F 0 "#PWR?" H 7350 3050 50  0001 C CNN
+F 0 "#PWR014" H 7350 3050 50  0001 C CNN
 F 1 "GND" H 7355 3127 50  0000 C CNN
 F 2 "" H 7350 3300 50  0001 C CNN
@@
 $EndComp
 $Comp
-L power:GND #PWR?
+L power:GND #PWR016
 U 1 1 60B49FFE
 P 7750 2850
-F 0 "#PWR?" H 7750 2600 50  0001 C CNN
+F 0 "#PWR016" H 7750 2600 50  0001 C CNN
 F 1 "GND" H 7755 2677 50  0000 C CNN
 F 2 "" H 7750 2850 50  0001 C CNN
@@
 $EndComp
 $Comp
-L power:GND #PWR?
+L power:GND #PWR08
 U 1 1 60B4A76D
 P 5050 4800
-F 0 "#PWR?" H 5050 4550 50  0001 C CNN
+F 0 "#PWR08" H 5050 4550 50  0001 C CNN
 F 1 "GND" H 5055 4627 50  0000 C CNN
 F 2 "" H 5050 4800 50  0001 C CNN
@@
 $EndComp
 $Comp
-L power:GND #PWR?
+L power:GND #PWR010
 U 1 1 60B4B142
 P 5750 4800
-F 0 "#PWR?" H 5750 4550 50  0001 C CNN
+F 0 "#PWR010" H 5750 4550 50  0001 C CNN
 F 1 "GND" H 5755 4627 50  0000 C CNN
 F 2 "" H 5750 4800 50  0001 C CNN
@@
 $EndComp
 $Comp
-L power:GND #PWR?
+L power:GND #PWR013
 U 1 1 60B4B8E1
 P 6450 4800
-F 0 "#PWR?" H 6450 4550 50  0001 C CNN
+F 0 "#PWR013" H 6450 4550 50  0001 C CNN
 F 1 "GND" H 6455 4627 50  0000 C CNN
 F 2 "" H 6450 4800 50  0001 C CNN

Commit message: Assign PCB footprints
Parts:
- C1, C2: footprint (none) -> Library:C_1206
- C3: footprint (none) -> Library:C_1210_Pad1.40x2.80mm
- C4, C5: footprint (none) -> Library:CP_2312
- D1: footprint (none) -> Library:LED_0805
- J1, J2: footprint (none) -> Library:Degson_15EDGRC-3.5
- L1: footprint (none) -> Library:L_TDK_RLF7030
- Q1: footprint Package_SO:SOIC-8_3.9x4.9mm_P1.27mm -> Library:SO-8
- R1, R2, R3, R4, R5: footprint (none) -> Library:R_1206
- SW1: footprint (none) -> Library:SW_Slide_CE_SL19121
- U1: footprint Package_SO:TI_SO-PowerPAD-8 -> Library:Power_SO-8
- U2: footprint (none) -> Library:SOT-223-4
Changed lines of the file:
@@
 F 0 "J1" H 2068 2167 50  0000 C CNN
 F 1 "Conn_01x02" H 2068 2076 50  0000 C CNN
-F 2 "" H 2150 1950 50  0001 C CNN
+F 2 "Library:Degson_15EDGRC-3.5" H 2150 1950 50  0001 C CNN
 F 3 "~" H 2150 1950 50  0001 C CNN
 	1    2150 1950
@@
 F 0 "J2" H 2068 2617 50  0000 C CNN
 F 1 "Conn_01x02" H 2068 2526 50  0000 C CNN
-F 2 "" H 2150 2400 50  0001 C CNN
+F 2 "Library:Degson_15EDGRC-3.5" H 2150 2400 50  0001 C CNN
 F 3 "~" H 2150 2400 50  0001 C CNN
 	1    2150 2400
@@
 F 0 "SW1" H 2800 2235 50  0000 C CNN
 F 1 "SW_SPDT" H 2800 2144 50  0000 C CNN
-F 2 "" H 2800 1950 50  0001 C CNN
+F 2 "Library:SW_Slide_CE_SL19121" H 2800 1950 50  0001 C CNN
 F 3 "~" H 2800 1950 50  0001 C CNN
 	1    2800 1950
@@
 F 0 "Q1" V 3642 2150 50  0000 C CNN
 F 1 "FDS4141" V 3551 2150 50  0000 C CNN
-F 2 "Package_SO:SOIC-8_3.9x4.9mm_P1.27mm" H 3500 2075 50  0001 L CIN
+F 2 "Library:SO-8" H 3500 2075 50  0001 L CIN
 F 3 "https://www.onsemi.com/pub/Collateral/FDS9435A-D.PDF" V 3300 2150 50  0001 L CNN
 	1    3300 2150
@@
 F 0 "R1" H 3670 2346 50  0000 L CNN
 F 1 "1k" H 3670 2255 50  0000 L CNN
-F 2 "" V 3530 2300 50  0001 C CNN
+F 2 "Library:R_1206" V 3530 2300 50  0001 C CNN
 F 3 "~" H 3600 2300 50  0001 C CNN
 	1    3600 2300
@@
 F 0 "R2" H 3670 2696 50  0000 L CNN
 F 1 "1k" H 3670 2605 50  0000 L CNN
-F 2 "" V 3530 2650 50  0001 C CNN
+F 2 "Library:R_1206" V 3530 2650 50  0001 C CNN
 F 3 "~" H 3600 2650 50  0001 C CNN
 	1    3600 2650
@@
 F 0 "D1" V 3639 2882 50  0000 R CNN
 F 1 "RED LED" V 3548 2882 50  0000 R CNN
-F 2 "" H 3600 3000 50  0001 C CNN
+F 2 "Library:LED_0805" H 3600 3000 50  0001 C CNN
 F 3 "~" H 3600 3000 50  0001 C CNN
 	1    3600 3000
@@
 F 0 "C1" H 5165 2646 50  0000 L CNN
 F 1 "4u7" H 5165 2555 50  0000 L CNN
-F 2 "" H 5088 2450 50  0001 C CNN
+F 2 "Library:C_1206" H 5088 2450 50  0001 C CNN
 F 3 "~" H 5050 2600 50  0001 C CNN
 	1    5050 2600
@@
 F 0 "C2" H 5565 2646 50  0000 L CNN
 F 1 "100n" H 5565 2555 50  0000 L CNN
-F 2 "" H 5488 2450 50  0001 C CNN
+F 2 "Library:C_1206" H 5488 2450 50  0001 C CNN
 F 3 "~" H 5450 2600 50  0001 C CNN
 	1    5450 2600
@@
 F 0 "U1" H 6400 2492 50  0000 C CNN
 F 1 "ST1S10PHR" H 6400 2401 50  0000 C CNN
-F 2 "Package_SO:TI_SO-PowerPAD-8" H 6525 1800 50  0001 L CIN
+F 2 "Library:Power_SO-8" H 6525 1800 50  0001 L CIN
 F 3 "http://www.st.com/internet/com/TECHNICAL_RESOURCES/TECHNICAL_LITERATURE/DATASHEET/CD00169322.pdf" H 6400 2150 50  0001 C CNN
 	1    6400 2150
@@
 F 0 "L1" V 7290 2050 50  0000 C CNN
 F 1 "3u3" V 7199 2050 50  0000 C CNN
-F 2 "" H 7100 2050 50  0001 C CNN
+F 2 "Library:L_TDK_RLF7030" H 7100 2050 50  0001 C CNN
 F 3 "~" H 7100 2050 50  0001 C CNN
 	1    7100 2050
@@
 F 0 "R3" H 7420 2346 50  0000 L CNN
 F 1 "100k" H 7420 2255 50  0000 L CNN
-F 2 "" V 7280 2300 50  0001 C CNN
+F 2 "Library:R_1206" V 7280 2300 50  0001 C CNN
 F 3 "~" H 7350 2300 50  0001 C CNN
 	1    7350 2300
@@
 F 0 "R4" H 7420 2696 50  0000 L CNN
 F 1 "5k1" H 7420 2605 50  0000 L CNN
-F 2 "" V 7280 2650 50  0001 C CNN
+F 2 "Library:R_1206" V 7280 2650 50  0001 C CNN
 F 3 "~" H 7350 2650 50  0001 C CNN
 	1    7350 2650
@@
 F 0 "R5" H 7420 3096 50  0000 L CNN
 F 1 "20k" H 7420 3005 50  0000 L CNN
-F 2 "" V 7280 3050 50  0001 C CNN
+F 2 "Library:R_1206" V 7280 3050 50  0001 C CNN
 F 3 "~" H 7350 3050 50  0001 C CNN
 	1    7350 3050
@@
 F 0 "C3" H 7865 2346 50  0000 L CNN
 F 1 "22u" H 7865 2255 50  0000 L CNN
-F 2 "" H 7788 2150 50  0001 C CNN
+F 2 "Library:C_1210_Pad1.40x2.80mm" H 7788 2150 50  0001 C CNN
 F 3 "~" H 7750 2300 50  0001 C CNN
 	1    7750 2300
@@
 F 0 "C4" H 5168 4596 50  0000 L CNN
 F 1 "10u" H 5168 4505 50  0000 L CNN
-F 2 "" H 5088 4400 50  0001 C CNN
+F 2 "Library:CP_2312" H 5088 4400 50  0001 C CNN
 F 3 "~" H 5050 4550 50  0001 C CNN
 	1    5050 4550
@@
 F 0 "U2" H 5750 4542 50  0000 C CNN
 F 1 "LM1117-3.3" H 5750 4451 50  0000 C CNN
-F 2 "" H 5750 4300 50  0001 C CNN
+F 2 "Library:SOT-223-4" H 5750 4300 50  0001 C CNN
 F 3 "http://www.ti.com/lit/ds/symlink/lm1117.pdf" H 5750 4300 50  0001 C CNN
 	1    5750 4300
@@
 F 0 "C5" H 6568 4596 50  0000 L CNN
 F 1 "10u" H 6568 4505 50  0000 L CNN
-F 2 "" H 6488 4400 50  0001 C CNN
+F 2 "Library:CP_2312" H 6488 4400 50  0001 C CNN
 F 3 "~" H 6450 4550 50  0001 C CNN
 	1    6450 4550
