File: wobbly.kicad_pcb (KiCad board)
At the start: 2 copper layers, 100 x 70 mm, 84 parts, among them J1 Conn_01x02, J10 Conn_01x14, J2 Conn_01x02, J3 Conn_02x03_Odd_Even, J4 Conn_01x06, J5 Conn_01x03, J6 Conn_01x04, J7 Conn_01x08, J8 Conn_01x04, J9 Conn_01x04, Q1 FDS4141, Q2 BSS138, Q3 BSS138, Q4 BSS138, Q5 BSS138, Q6 BSS138, SW1 SW_SPDT, SW2 SW_Push, SW3 SW_Push, U1 ST1S10PHR, U2 LM1117, U3 ATmega324PB-AU, U4 74LVC1G58, U5 74LVC1G58, Y1 Crystal

Commit message: Add graphics
Parts:
- added G1: LOGO, Wobbly:wobbly_logo, F.Cu at (48.9, 73.0)
- added G10: RST, Wobbly:rst, F.Cu at (111.1, 94.2)
- added G11: BATT, Wobbly:batt, B.Cu at (36.3, 45.3)
- added G12: VSW, Wobbly:vsw, B.Cu at (36.3, 56.3)
- added G13: PWR SW, Wobbly:pwr_sw, B.Cu at (35.7, 29.6)
- added G14: IMU, Wobbly:imu, B.Cu at (64.3, 30.1)
- added G15: BT, Wobbly:bt, B.Cu at (105.5, 30.1)
- added G16: DRV, Wobbly:drv, B.Cu at (74.3, 58.7)
- added G17: ENC R, Wobbly:enc_r, B.Cu at (91.3, 58.7)
- added G18: ENC L, Wobbly:enc_l, B.Cu at (104.1, 58.7)
- added G2: VERSION, Wobbly:version, F.Cu at (61.3, 76.8)
- added G3: EXT, Wobbly:ext, F.Cu at (66.9, 67.6)
- added G4: PWR, Wobbly:pwr, F.Cu at (39.4, 94.2)
- added G5: STATE, Wobbly:state, F.Cu at (47.0, 94.2)
- added G6: CONN, Wobbly:conn, F.Cu at (54.6, 94.2)
- added G7: SIG, Wobbly:sig, F.Cu at (62.2, 94.2)
- added G8: FUN, Wobbly:fun, F.Cu at (74.3, 94.2)
- added G9: ISP, Wobbly:isp, F.Cu at (95.0, 94.2)
- moved D1 1.27 mm to (39.4, 90.2)
- moved D2 1.27 mm to (47.0, 90.2)
- moved D3 1.27 mm to (54.6, 90.2)
- moved D4 1.27 mm to (62.2, 90.2)
Routing:
- net Net-(D4-Pad2): track 6.38 -> 5.11 mm
- net Net-(D3-Pad2): track 6.38 -> 5.11 mm
- net Net-(D2-Pad2): track 6.38 -> 5.11 mm
- net Net-(D1-Pad2): track 6.38 -> 5.11 mm
Other:
- board text removed: "BAT"
- board text removed: "BT"
- board text removed: "ENC L"
- board text removed: "ENC R"
- board text removed: "EXT"
- board text removed: "FUN"
- board text removed: "IMU"
- board text removed: "ISP"
- board text removed: "MOTOR"
- board text removed: "MOTOR DRV"
- board text removed: "PWR"
- board text removed: "PWR SW"
- board text removed: "RST"
- board text removed: "SIG"
- board text removed: "STATE"
